File: controle.kicad_sch (KiCad schematic)
At the start: 7 parts, among them J4 USB_B, J5 Conn_01x03, J6 Conn_01x04, U2 ProMicroC, U4 6N137, U5 6N137

Commit message: alteração no circuito de controle: adição dos isoladores
  Changes to be committed:
 	new file:   .history
 	modified:   controle.kicad_sch
 	modified:   dc_converter_sch.kicad_sch
 	modified:   h_bridge_sch.kicad_sch
 	modified:   half_bridge.kicad_sch
 	modified:   volante.kicad_pcb
 	modified:   volante.kicad_prl
 	modified:   volante.kicad_pro
 	modified:   volante.kicad_sch

  Changes not staged for commit:
 	modified:   .history (modified content, untracked content)
Parts:
- U3: value ~ -> (none)
