File: dc_converter_sch.kicad_sch (KiCad schematic)
At the start: 8 parts, among them J1 ATX-24, J2 Conn_01x02_Pin, U1 AP3012

Commit message: foi adicionado o arduino e conector de encoder na mesma placa, utilizando optacopladores recomeço do layout pcb
 Changes to be committed:
	new file:   controle.kicad_sch
	modified:   dc_converter_sch.kicad_sch
	modified:   half_bridge.kicad_sch
	modified:   volante.kicad_pcb
	modified:   volante.kicad_prl
	modified:   volante.kicad_pro
	modified:   volante.kicad_sch
Parts:
- C1, D1, L1, R1, R2, U1: now left out of the parts list
Connections:
- net V22: no longer C1.1, D1.1 (K), R1.1
- new net: C1.1, D1.1 (K), R1.1
Other:
- moved on the sheet: C1, D1, L1, R1, R2, U1
